Commit message: Fix mesh paths, update thymio model and sensors

File: thymio_description/thymio/urdf/base.urdf.xacro (robot description, xacro)
@@ -27,4 +27,26 @@
   </xacro:if>
   <xacro:macro name="thymio">
+      <link name="${tf_prefix}camera_link">
+      <inertial>
+        <origin xyz="0 0 0"/>
+        <mass value="0.01"/>
+        <inertia ixx="1e-6" ixy="0" ixz="0" iyy="1e-6" iyz="0" izz="1e-6"/>
+      </inertial>
+      <visual>
+        <geometry>
+          <box size="0.02 0.02 0.02"/>
+        </geometry>
+      </visual>
+      <collision>
+        <geometry>
+          <box size="0.02 0.02 0.02"/>
+        </geometry>
+      </collision>
+    </link>
+    <joint name="${tf_prefix}camera_joint" type="fixed">
+      <parent link="${tf_prefix}base_link"/>
+      <child link="${tf_prefix}camera_link"/>
+      <origin xyz="0.05 0 0.1" rpy="0 0 0"/>
+    </joint>
     <link name="${tf_prefix}base_link">
       <collision>
@@ -81,4 +103,31 @@
       <origin xyz="0 0 0.035"/>
     </joint>
+    <gazebo reference="${tf_prefix}camera_link">
+      <sensor type="camera" name="${tf_prefix}camera_sensor">
+        <always_on>true</always_on>
+        <update_rate>10.0</update_rate>
+        <visualize>true</visualize>
+        <camera>
+          <horizontal_fov>1.047</horizontal_fov>
+          <image>
+            <width>1920</width>
+            <height>1080</height>
+            <format>R8G8B8</format>
+          </image>
+          <clip>
+            <near>0.05</near>
+            <far>10.0</far>
+          </clip>
+        </camera>
+        <plugin name="${_name}_camera_controller" filename="libgazebo_ros_camera.so">
+          <frame_name>${tf_prefix}camera_link</frame_name>
+          <ros>
+            <namespace>${_name}</namespace>
+            <remapping>image_raw:=camera/image_raw</remapping>
+            <remapping>camera_info:=camera/camera_info</remapping>
+          </ros>
+        </plugin>
+      </sensor>
+    </gazebo>
     <!-- We have a problem with xacro -->
     <!-- <xacro:imu ns="$(arg name)"/> -->

File: thymio_description/thymio/urdf/proximity_sensor.urdf.xacro (robot description, xacro)
@@ -20,11 +20,11 @@
               <resolution>1</resolution>
               <min_angle>-${fov / 2}</min_angle>
-              <max_angle>-${fov / 2}</max_angle>
+              <max_angle>${fov / 2}</max_angle>
             </horizontal>
             <vertical>
               <samples>1</samples>
               <resolution>1</resolution>
-              <min_angle>-${fov / 2}</min_angle>
-              <max_angle>-${fov / 2}</max_angle>
+              <min_angle>0</min_angle>
+              <max_angle>0</max_angle>
             </vertical>
           </scan>
@@ -41,5 +41,4 @@
         </ray>
         <plugin name="${group}_${name}_controller" filename="libgazebo_ros_ray_sensor.so">
-          <!-- TODO: check if field `radiation` is still valid-->
           <radiation_type>infrared</radiation_type>
           <ros>
@@ -47,5 +46,5 @@
             <argument>~/out:=${group}/${name}</argument>
           </ros>
-          <output_type>sensor_msgs/Range</output_type>
+          <output_type>sensor_msgs/LaserScan</output_type>
         </plugin>
       </sensor>

Commit message: basic nn controller + training cycles, gazebo crashes, will try to switch to argos

File: thymio_description/thymio/urdf/base.urdf.xacro (robot description, xacro)
@@ -5,4 +5,5 @@
   <xacro:include filename="imu.urdf.xacro"/>
   <xacro:arg name="name" default="thymio2"/>
+  <xacro:arg name="body_color" default="Gazebo/White"/>
   <xacro:arg name="left_wheel_mu" default="100.0"/>
   <xacro:arg name="right_wheel_mu" default="100.0"/>
@@ -35,10 +36,10 @@
       <visual>
         <geometry>
-          <box size="0.02 0.02 0.02"/>
+          <box size="0.01 0.01 0.01"/>
         </geometry>
       </visual>
       <collision>
         <geometry>
-          <box size="0.02 0.02 0.02"/>
+          <box size="0.01 0.01 0.01"/>
         </geometry>
       </collision>
@@ -47,5 +48,5 @@
       <parent link="${tf_prefix}base_link"/>
       <child link="${tf_prefix}camera_link"/>
-      <origin xyz="0.05 0 0.1" rpy="0 0 0"/>
+      <origin xyz="0.075 0 0.045" rpy="0 0 0"/>
     </joint>
     <link name="${tf_prefix}base_link">
@@ -85,4 +86,5 @@
       <mu1>0.1</mu1>
       <mu2>0.1</mu2>
+      <material>$(arg body_color)</material>
     </gazebo>
     <xacro:wheel tf_prefix="${tf_prefix}" name="left" position="${wheel_axis * 0.5}" radius="${wheel_radius}" mass="${wheel_mass}" mu="$(arg left_wheel_mu)"/>
@@ -104,13 +106,13 @@
     </joint>
     <gazebo reference="${tf_prefix}camera_link">
-      <sensor type="camera" name="${tf_prefix}camera_sensor">
+      <sensor type="camera" name="camera_sensor">
         <always_on>true</always_on>
-        <update_rate>10.0</update_rate>
-        <visualize>true</visualize>
+        <update_rate>5.0</update_rate>
+        <visualize>false</visualize>
         <camera>
           <horizontal_fov>1.047</horizontal_fov>
           <image>
-            <width>1920</width>
-            <height>1080</height>
+            <width>320</width>
+            <height>240</height>
             <format>R8G8B8</format>
           </image>

Commit message: Fixed sensor read problem, fitness function seems to work, but needs to be modified

File: thymio_description/thymio/urdf/base.urdf.xacro (robot description, xacro)
@@ -63,4 +63,10 @@
         </geometry>
       </collision>
+      <collision name="front_bottom_bumper_collision">
+        <origin xyz="0.086 0 0.012" rpy="0 0 0"/>
+        <geometry>
+          <box size="0.018 0.090 0.018"/>
+        </geometry>
+      </collision>
       <visual>
         <origin xyz="0.0 0 0.0" rpy="0 0 0"/>
@@ -108,5 +114,5 @@
       <sensor type="camera" name="camera_sensor">
         <always_on>true</always_on>
-        <update_rate>5.0</update_rate>
+        <update_rate>$(arg odom_rate)</update_rate>
         <visualize>false</visualize>
         <camera>

Commit message: robot description updated to use 360 camera(4*90), this robot will be used in all 3 experiments so structuresays clear

File: thymio_description/thymio/urdf/base.urdf.xacro (robot description, xacro)
@@ -28,5 +28,5 @@
   </xacro:if>
   <xacro:macro name="thymio">
-      <link name="${tf_prefix}camera_link">
+      <link name="${tf_prefix}camera_front_link">
       <inertial>
         <origin xyz="0 0 0"/>
@@ -36,10 +36,10 @@
       <visual>
         <geometry>
-          <box size="0.01 0.01 0.01"/>
-        </geometry>
-      </visual>
-      <collision>
-        <geometry>
-          <box size="0.01 0.01 0.01"/>
+          <box size="0.015 0.015 0.015"/>
+        </geometry>
+      </visual>
+      <collision>
+        <geometry>
+          <box size="0.001 0.001 0.001"/>
         </geometry>
       </collision>
@@ -47,6 +47,78 @@
     <joint name="${tf_prefix}camera_joint" type="fixed">
       <parent link="${tf_prefix}base_link"/>
-      <child link="${tf_prefix}camera_link"/>
-      <origin xyz="0.075 0 0.045" rpy="0 0 0"/>
+      <child link="${tf_prefix}camera_front_link"/>
+      <origin xyz="0.025 0.000 0.100" rpy="0 0 0"/>
+    </joint>
+    <!-- Cameras for simulated 360-degree perception.
+         All four cameras are mounted above the robot at the same height.
+         The front camera keeps its existing topic for FPV compatibility.
+         Privileged controllers ignore all cameras.
+         FPV controllers use only the front camera.
+         360 controllers use front + left + right + rear cameras. -->
+    <link name="${tf_prefix}camera_left_link">
+      <inertial>
+        <origin xyz="0 0 0"/>
+        <mass value="0.01"/>
+        <inertia ixx="1e-6" ixy="0" ixz="0" iyy="1e-6" iyz="0" izz="1e-6"/>
+      </inertial>
+      <visual>
+        <geometry>
+          <box size="0.015 0.015 0.015"/>
+        </geometry>
+      </visual>
+      <collision>
+        <geometry>
+          <box size="0.001 0.001 0.001"/>
+        </geometry>
+      </collision>
+    </link>
+    <joint name="${tf_prefix}camera_left_joint" type="fixed">
+      <parent link="${tf_prefix}base_link"/>
+      <child link="${tf_prefix}camera_left_link"/>
+      <origin xyz="0.025 0.000 0.100" rpy="0 0 1.5708"/>
+    </joint>
+    <link name="${tf_prefix}camera_right_link">
+      <inertial>
+        <origin xyz="0 0 0"/>
+        <mass value="0.01"/>
+        <inertia ixx="1e-6" ixy="0" ixz="0" iyy="1e-6" iyz="0" izz="1e-6"/>
+      </inertial>
+      <visual>
+        <geometry>
+          <box size="0.015 0.015 0.015"/>
+        </geometry>
+      </visual>
+      <collision>
+        <geometry>
+          <box size="0.001 0.001 0.001"/>
+        </geometry>
+      </collision>
+    </link>
+    <joint name="${tf_prefix}camera_right_joint" type="fixed">
+      <parent link="${tf_prefix}base_link"/>
+      <child link="${tf_prefix}camera_right_link"/>
+      <origin xyz="0.025 0.000 0.100" rpy="0 0 -1.5708"/>
+    </joint>
+    <link name="${tf_prefix}camera_rear_link">
+      <inertial>
+        <origin xyz="0 0 0"/>
+        <mass value="0.01"/>
+        <inertia ixx="1e-6" ixy="0" ixz="0" iyy="1e-6" iyz="0" izz="1e-6"/>
+      </inertial>
+      <visual>
+        <geometry>
+          <box size="0.015 0.015 0.015"/>
+        </geometry>
+      </visual>
+      <collision>
+        <geometry>
+          <box size="0.001 0.001 0.001"/>
+        </geometry>
+      </collision>
+    </link>
+    <joint name="${tf_prefix}camera_rear_joint" type="fixed">
+      <parent link="${tf_prefix}base_link"/>
+      <child link="${tf_prefix}camera_rear_link"/>
+      <origin xyz="0.025 0.000 0.100" rpy="0 0 3.14159"/>
     </joint>
     <link name="${tf_prefix}base_link">
@@ -111,11 +183,11 @@
       <origin xyz="0 0 0.035"/>
     </joint>
-    <gazebo reference="${tf_prefix}camera_link">
-      <sensor type="camera" name="camera_sensor">
-        <always_on>true</always_on>
-        <update_rate>$(arg odom_rate)</update_rate>
-        <visualize>false</visualize>
+    <gazebo reference="${tf_prefix}camera_front_link">
+      <sensor type="camera" name="camera_front_sensor">
+        <always_on>true</always_on>
+        <update_rate>$(arg odom_rate)</update_rate>
+        <visualize>true</visualize>
         <camera>
-          <horizontal_fov>1.047</horizontal_fov>
+          <horizontal_fov>1.5708</horizontal_fov>
           <image>
             <width>320</width>
@@ -129,9 +201,90 @@
         </camera>
         <plugin name="${_name}_camera_controller" filename="libgazebo_ros_camera.so">
-          <frame_name>${tf_prefix}camera_link</frame_name>
+          <frame_name>${tf_prefix}camera_front_link</frame_name>
           <ros>
             <namespace>${_name}</namespace>
             <remapping>image_raw:=camera/image_raw</remapping>
             <remapping>camera_info:=camera/camera_info</remapping>
+          </ros>
+        </plugin>
+      </sensor>
+    </gazebo>
+    <gazebo reference="${tf_prefix}camera_left_link">
+      <sensor type="camera" name="camera_left_sensor">
+        <always_on>true</always_on>
+        <update_rate>$(arg odom_rate)</update_rate>
+        <visualize>true</visualize>
+        <camera>
+          <horizontal_fov>1.5708</horizontal_fov>
+          <image>
+            <width>320</width>
+            <height>240</height>
+            <format>R8G8B8</format>
+          </image>
+          <clip>
+            <near>0.05</near>
+            <far>10.0</far>
+          </clip>
+        </camera>
+        <plugin name="${_name}_camera_left_controller" filename="libgazebo_ros_camera.so">
+          <frame_name>${tf_prefix}camera_left_link</frame_name>
+          <ros>
+            <namespace>${_name}</namespace>
+            <remapping>image_raw:=camera_left/image_raw</remapping>
+            <remapping>camera_info:=camera_left/camera_info</remapping>
+          </ros>
+        </plugin>
+      </sensor>
+    </gazebo>
+    <gazebo reference="${tf_prefix}camera_right_link">
+      <sensor type="camera" name="camera_right_sensor">
+        <always_on>true</always_on>
+        <update_rate>$(arg odom_rate)</update_rate>
+        <visualize>true</visualize>
+        <camera>
+          <horizontal_fov>1.5708</horizontal_fov>
+          <image>
+            <width>320</width>
+            <height>240</height>
+            <format>R8G8B8</format>
+          </image>
+          <clip>
+            <near>0.05</near>
+            <far>10.0</far>
+          </clip>
+        </camera>
+        <plugin name="${_name}_camera_right_controller" filename="libgazebo_ros_camera.so">
+          <frame_name>${tf_prefix}camera_right_link</frame_name>
+          <ros>
+            <namespace>${_name}</namespace>
+            <remapping>image_raw:=camera_right/image_raw</remapping>
+            <remapping>camera_info:=camera_right/camera_info</remapping>
+          </ros>
+        </plugin>
+      </sensor>
+    </gazebo>
+    <gazebo reference="${tf_prefix}camera_rear_link">
+      <sensor type="camera" name="camera_rear_sensor">
+        <always_on>true</always_on>
+        <update_rate>$(arg odom_rate)</update_rate>
+        <visualize>true</visualize>
+        <camera>
+          <horizontal_fov>1.5708</horizontal_fov>
+          <image>
+            <width>320</width>
+            <height>240</height>
+            <format>R8G8B8</format>
+          </image>
+          <clip>
+            <near>0.05</near>
+            <far>10.0</far>
+          </clip>
+        </camera>
+        <plugin name="${_name}_camera_rear_controller" filename="libgazebo_ros_camera.so">
+          <frame_name>${tf_prefix}camera_rear_link</frame_name>
+          <ros>
+            <namespace>${_name}</namespace>
+            <remapping>image_raw:=camera_rear/image_raw</remapping>
+            <remapping>camera_info:=camera_rear/camera_info</remapping>
           </ros>
         </plugin>
