Commit message: use simulation time, not real time, x3 speed now, change policies and change observation code

File: thymio_description/thymio/urdf/base.urdf.xacro (robot description, xacro)
@@ -1,11 +1,19 @@
 <?xml version="1.0"?>
 <robot xmlns:xacro="http://playerstage.sourceforge.net/gazebo/xmlschema/#xacro" name="thymio">
+  <!-- Cleaned thesis version:
+       - keeps wheels / differential drive
+       - keeps front, left, right, rear cameras for FPV and 360 experiments
+       - keeps optional ground-truth odometry for fitness, prey, and privileged observation
+       - removes proximity sensors, ground sensors, IMU include, and unused laser link
+  -->
   <xacro:include filename="wheel.urdf.xacro"/>
-  <xacro:include filename="proximity_sensor.urdf.xacro"/>
-  <xacro:include filename="imu.urdf.xacro"/>
   <xacro:arg name="name" default="thymio2"/>
   <xacro:arg name="body_color" default="Gazebo/White"/>
   <xacro:arg name="left_wheel_mu" default="100.0"/>
   <xacro:arg name="right_wheel_mu" default="100.0"/>
+  <xacro:arg name="publish_ground_truth" default="false"/>
+  <xacro:arg name="ground_truth_frame_id" default="/world"/>
+  <xacro:arg name="ground_truth_update_rate" default="10.0"/>
+  <xacro:arg name="odom_rate" default="20.0"/>
   <xacro:property name="wheel_axis" value="0.0935"/>
   <xacro:property name="wheel_radius" value="0.022"/>
@@ -13,11 +21,4 @@
   <xacro:property name="body_mass" value="0.2"/>
   <xacro:property name="wheel_mass" value="0.024"/>
-  <xacro:arg name="proximity_max_range" default="0.12"/>
-  <xacro:arg name="proximity_resolution" default="0.005"/>
-  <xacro:arg name="proximity_fov" default="0.3"/>
-  <xacro:arg name="publish_ground_truth" default="false"/>
-  <xacro:arg name="ground_truth_frame_id" default="/world"/>
-  <xacro:arg name="ground_truth_update_rate" default="10.0"/>
-  <xacro:arg name="odom_rate" default="20.0"/>
   <xacro:property name="_name" value="$(arg name)"/>
   <xacro:if value="${_name != ''}">
@@ -27,6 +28,6 @@
     <xacro:property name="tf_prefix" value=""/>
   </xacro:if>
-  <xacro:macro name="thymio">
-      <link name="${tf_prefix}camera_front_link">
+  <xacro:macro name="camera_link" params="suffix xyz rpy">
+    <link name="${tf_prefix}camera_${suffix}_link">
       <inertial>
         <origin xyz="0 0 0"/>
@@ -34,92 +35,41 @@
         <inertia ixx="1e-6" ixy="0" ixz="0" iyy="1e-6" iyz="0" izz="1e-6"/>
       </inertial>
-      <visual>
-        <geometry>
-          <box size="0.015 0.015 0.015"/>
-        </geometry>
-      </visual>
-      <collision>
-        <geometry>
-          <box size="0.001 0.001 0.001"/>
-        </geometry>
-      </collision>
     </link>
-    <joint name="${tf_prefix}camera_joint" type="fixed">
+    <joint name="${tf_prefix}camera_${suffix}_joint" type="fixed">
       <parent link="${tf_prefix}base_link"/>
-      <child link="${tf_prefix}camera_front_link"/>
-      <origin xyz="0.025 0.000 0.100" rpy="0 0 0"/>
+      <child link="${tf_prefix}camera_${suffix}_link"/>
+      <origin xyz="${xyz}" rpy="${rpy}"/>
     </joint>
-    <!-- Cameras for simulated 360-degree perception.
-         All four cameras are mounted above the robot at the same height.
-         The front camera keeps its existing topic for FPV compatibility.
-         Privileged controllers ignore all cameras.
-         FPV controllers use only the front camera.
-         360 controllers use front + left + right + rear cameras. -->
-    <link name="${tf_prefix}camera_left_link">
-      <inertial>
-        <origin xyz="0 0 0"/>
-        <mass value="0.01"/>
-        <inertia ixx="1e-6" ixy="0" ixz="0" iyy="1e-6" iyz="0" izz="1e-6"/>
-      </inertial>
-      <visual>
-        <geometry>
-          <box size="0.015 0.015 0.015"/>
-        </geometry>
-      </visual>
-      <collision>
-        <geometry>
-          <box size="0.001 0.001 0.001"/>
-        </geometry>
-      </collision>
-    </link>
-    <joint name="${tf_prefix}camera_left_joint" type="fixed">
-      <parent link="${tf_prefix}base_link"/>
-      <child link="${tf_prefix}camera_left_link"/>
-      <origin xyz="0.025 0.000 0.100" rpy="0 0 1.5708"/>
-    </joint>
-    <link name="${tf_prefix}camera_right_link">
-      <inertial>
-        <origin xyz="0 0 0"/>
-        <mass value="0.01"/>
-        <inertia ixx="1e-6" ixy="0" ixz="0" iyy="1e-6" iyz="0" izz="1e-6"/>
-      </inertial>
-      <visual>
-        <geometry>
-          <box size="0.015 0.015 0.015"/>
-        </geometry>
-      </visual>
-      <collision>
-        <geometry>
-          <box size="0.001 0.001 0.001"/>
-        </geometry>
-      </collision>
-    </link>
-    <joint name="${tf_prefix}camera_right_joint" type="fixed">
-      <parent link="${tf_prefix}base_link"/>
-      <child link="${tf_prefix}camera_right_link"/>
-      <origin xyz="0.025 0.000 0.100" rpy="0 0 -1.5708"/>
-    </joint>
-    <link name="${tf_prefix}camera_rear_link">
-      <inertial>
-        <origin xyz="0 0 0"/>
-        <mass value="0.01"/>
-        <inertia ixx="1e-6" ixy="0" ixz="0" iyy="1e-6" iyz="0" izz="1e-6"/>
-      </inertial>
-      <visual>
-        <geometry>
-          <box size="0.015 0.015 0.015"/>
-        </geometry>
-      </visual>
-      <collision>
-        <geometry>
-          <box size="0.001 0.001 0.001"/>
-        </geometry>
-      </collision>
-    </link>
-    <joint name="${tf_prefix}camera_rear_joint" type="fixed">
-      <parent link="${tf_prefix}base_link"/>
-      <child link="${tf_prefix}camera_rear_link"/>
-      <origin xyz="0.025 0.000 0.100" rpy="0 0 3.14159"/>
-    </joint>
+  </xacro:macro>
+  <xacro:macro name="camera_sensor" params="suffix topic">
+    <gazebo reference="${tf_prefix}camera_${suffix}_link">
+      <sensor type="camera" name="camera_${suffix}_sensor">
+        <always_on>true</always_on>
+        <update_rate>$(arg odom_rate)</update_rate>
+        <visualize>false</visualize>
+        <camera>
+          <horizontal_fov>1.5708</horizontal_fov>
+          <image>
+            <width>320</width>
+            <height>240</height>
+            <format>R8G8B8</format>
+          </image>
+          <clip>
+            <near>0.05</near>
+            <far>10.0</far>
+          </clip>
+        </camera>
+        <plugin name="${_name}_camera_${suffix}_controller" filename="libgazebo_ros_camera.so">
+          <frame_name>${tf_prefix}camera_${suffix}_link</frame_name>
+          <ros>
+            <namespace>${_name}</namespace>
+            <remapping>image_raw:=${topic}/image_raw</remapping>
+            <remapping>camera_info:=${topic}/camera_info</remapping>
+          </ros>
+        </plugin>
+      </sensor>
+    </gazebo>
+  </xacro:macro>
+  <xacro:macro name="thymio">
     <link name="${tf_prefix}base_link">
       <collision>
@@ -133,10 +83,4 @@
         <geometry>
           <sphere radius="0.009"/>
-        </geometry>
-      </collision>
-      <collision name="front_bottom_bumper_collision">
-        <origin xyz="0.086 0 0.012" rpy="0 0 0"/>
-        <geometry>
-          <box size="0.018 0.090 0.018"/>
         </geometry>
       </collision>
@@ -168,130 +112,13 @@
     <xacro:wheel tf_prefix="${tf_prefix}" name="left" position="${wheel_axis * 0.5}" radius="${wheel_radius}" mass="${wheel_mass}" mu="$(arg left_wheel_mu)"/>
     <xacro:wheel tf_prefix="${tf_prefix}" name="right" position="${-wheel_axis * 0.5}" radius="${wheel_radius}" mass="${wheel_mass}" mu="$(arg right_wheel_mu)"/>
-    <xacro:proximity_sensor ns="${_name}" tf_prefix="${tf_prefix}" group="proximity" range_max="$(arg proximity_max_range)" resolution="$(arg proximity_resolution)" fov="$(arg proximity_fov)" name="center" xyz="0.0805 0 0.035" rpy="0 0 0"/>
-    <xacro:proximity_sensor ns="${_name}" tf_prefix="${tf_prefix}" group="proximity" range_max="$(arg proximity_max_range)" resolution="$(arg proximity_resolution)" fov="$(arg proximity_fov)" name="center_left" xyz="0.0756 0.0261 0.035" rpy="0 0 0.33161"/>
-    <xacro:proximity_sensor ns="${_name}" tf_prefix="${tf_prefix}" group="proximity" range_max="$(arg proximity_max_range)" resolution="$(arg proximity_resolution)" fov="$(arg proximity_fov)" name="center_right" xyz="0.0756 -0.0261 0.035" rpy="0 0 -0.33161"/>
-    <xacro:proximity_sensor ns="${_name}" tf_prefix="${tf_prefix}" group="proximity" range_max="$(arg proximity_max_range)" resolution="$(arg proximity_resolution)" fov="$(arg proximity_fov)" name="left" xyz="0.063 0.0493 0.035" rpy="0 0 0.66323"/>
-    <xacro:proximity_sensor ns="${_name}" tf_prefix="${tf_prefix}" group="proximity" range_max="$(arg proximity_max_range)" resolution="$(arg proximity_resolution)" fov="$(arg proximity_fov)" name="right" xyz="0.063 -0.0493 0.035" rpy="0 0 -0.66323"/>
-    <xacro:proximity_sensor ns="${_name}" tf_prefix="${tf_prefix}" group="proximity" range_max="$(arg proximity_max_range)" resolution="$(arg proximity_resolution)" fov="$(arg proximity_fov)" name="rear_left" xyz="-0.0301 0.0305 0.035" rpy="0 0 3.14159"/>
-    <xacro:proximity_sensor ns="${_name}" tf_prefix="${tf_prefix}" group="proximity" range_max="$(arg proximity_max_range)" resolution="$(arg proximity_resolution)" fov="$(arg proximity_fov)" name="rear_right" xyz="-0.0301 -0.0305 0.035" rpy="0 0 3.14159"/>
-    <xacro:proximity_sensor ns="${_name}" tf_prefix="${tf_prefix}" group="ground" range_max="0.03" name="left" xyz="0.07157 0.01155 0.009" rpy="0 1.5708 0.24311"/>
-    <xacro:proximity_sensor ns="${_name}" tf_prefix="${tf_prefix}" group="ground" range_max="0.03" name="right" xyz="0.07157 -0.01155 0.009" rpy="0 1.5708 -0.24311"/>
-    <link name="${tf_prefix}laser_link"/>
-    <joint name="${tf_prefix}base_laser_joint" type="fixed">
-      <parent link="${tf_prefix}base_link"/>
-      <child link="${tf_prefix}laser_link"/>
-      <origin xyz="0 0 0.035"/>
-    </joint>
-    <gazebo reference="${tf_prefix}camera_front_link">
-      <sensor type="camera" name="camera_front_sensor">
-        <always_on>true</always_on>
-        <update_rate>$(arg odom_rate)</update_rate>
-        <visualize>false</visualize>
-        <camera>
-          <horizontal_fov>1.5708</horizontal_fov>
-          <image>
-            <width>320</width>
-            <height>240</height>
-            <format>R8G8B8</format>
-          </image>
-          <clip>
-            <near>0.05</near>
-            <far>10.0</far>
-          </clip>
-        </camera>
-        <plugin name="${_name}_camera_controller" filename="libgazebo_ros_camera.so">
-          <frame_name>${tf_prefix}camera_front_link</frame_name>
-          <ros>
-            <namespace>${_name}</namespace>
-            <remapping>image_raw:=camera/image_raw</remapping>
-            <remapping>camera_info:=camera/camera_info</remapping>
-          </ros>
-        </plugin>
-      </sensor>
-    </gazebo>
-    <gazebo reference="${tf_prefix}camera_left_link">
-      <sensor type="camera" name="camera_left_sensor">
-        <always_on>true</always_on>
-        <update_rate>$(arg odom_rate)</update_rate>
-        <visualize>false</visualize>
-        <camera>
-          <horizontal_fov>1.5708</horizontal_fov>
-          <image>
-            <width>320</width>
-            <height>240</height>
-            <format>R8G8B8</format>
-          </image>
-          <clip>
-            <near>0.05</near>
-            <far>10.0</far>
-          </clip>
-        </camera>
-        <plugin name="${_name}_camera_left_controller" filename="libgazebo_ros_camera.so">
-          <frame_name>${tf_prefix}camera_left_link</frame_name>
-          <ros>
-            <namespace>${_name}</namespace>
-            <remapping>image_raw:=camera_left/image_raw</remapping>
-            <remapping>camera_info:=camera_left/camera_info</remapping>
-          </ros>
-        </plugin>
-      </sensor>
-    </gazebo>
-    <gazebo reference="${tf_prefix}camera_right_link">
-      <sensor type="camera" name="camera_right_sensor">
-        <always_on>true</always_on>
-        <update_rate>$(arg odom_rate)</update_rate>
-        <visualize>false</visualize>
-        <camera>
-          <horizontal_fov>1.5708</horizontal_fov>
-          <image>
-            <width>320</width>
-            <height>240</height>
-            <format>R8G8B8</format>
-          </image>
-          <clip>
-            <near>0.05</near>
-            <far>10.0</far>
-          </clip>
-        </camera>
-        <plugin name="${_name}_camera_right_controller" filename="libgazebo_ros_camera.so">
-          <frame_name>${tf_prefix}camera_right_link</frame_name>
-          <ros>
-            <namespace>${_name}</namespace>
-            <remapping>image_raw:=camera_right/image_raw</remapping>
-            <remapping>camera_info:=camera_right/camera_info</remapping>
-          </ros>
-        </plugin>
-      </sensor>
-    </gazebo>
-    <gazebo reference="${tf_prefix}camera_rear_link">
-      <sensor type="camera" name="camera_rear_sensor">
-        <always_on>true</always_on>
-        <update_rate>$(arg odom_rate)</update_rate>
-        <visualize>false</visualize>
-        <camera>
-          <horizontal_fov>1.5708</horizontal_fov>
-          <image>
-            <width>320</width>
-            <height>240</height>
-            <format>R8G8B8</format>
-          </image>
-          <clip>
-            <near>0.05</near>
-            <far>10.0</far>
-          </clip>
-        </camera>
-        <plugin name="${_name}_camera_rear_controller" filename="libgazebo_ros_camera.so">
-          <frame_name>${tf_prefix}camera_rear_link</frame_name>
-          <ros>
-            <namespace>${_name}</namespace>
-            <remapping>image_raw:=camera_rear/image_raw</remapping>
-            <remapping>camera_info:=camera_rear/camera_info</remapping>
-          </ros>
-        </plugin>
-      </sensor>
-    </gazebo>
-    <!-- We have a problem with xacro -->
-    <!-- <xacro:imu ns="$(arg name)"/> -->
-    <!-- see https://github.com/ros-simulation/gazebo_ros_pkgs/blob/kinetic-devel/gazebo_plugins/src/gazebo_ros_diff_drive.cpp -->
+    <!-- Cameras: front is also remapped to /<robot>/camera/image_raw for FPV compatibility. -->
+    <xacro:camera_link suffix="front" xyz="0.025 0.000 0.100" rpy="0 0 0"/>
+    <xacro:camera_link suffix="left" xyz="0.025 0.000 0.100" rpy="0 0 1.5708"/>
+    <xacro:camera_link suffix="right" xyz="0.025 0.000 0.100" rpy="0 0 -1.5708"/>
+    <xacro:camera_link suffix="rear" xyz="0.025 0.000 0.100" rpy="0 0 3.14159"/>
+    <xacro:camera_sensor suffix="front" topic="camera"/>
+    <xacro:camera_sensor suffix="left" topic="camera_left"/>
+    <xacro:camera_sensor suffix="right" topic="camera_right"/>
+    <xacro:camera_sensor suffix="rear" topic="camera_rear"/>
     <gazebo>
       <plugin name="differential_drive_controller" filename="libgazebo_ros_diff_drive.so">
@@ -319,13 +146,8 @@
       </plugin>
     </gazebo>
-    <!-- NOTE: The current version of the gazebo p3d plugin has a bug:
-    the field child_frame_id is set to the name of the link (bodyName)
-    and not to the frame name (frameName). -->
     <xacro:if value="$(arg publish_ground_truth)">
       <gazebo>
         <plugin name="ground_truth" filename="libgazebo_ros_p3d.so">
           <ros>
-            <!-- Add namespace and remap the default topic -->
-            <!-- TODO namespace is ignored! -->
             <namespace>${_name}</namespace>
             <argument>odom:=ground_truth/odom</argument>
@@ -336,5 +158,5 @@
         </plugin>
       </gazebo>
-     </xacro:if>
+    </xacro:if>
   </xacro:macro>
 </robot>
